Commit message: tb3_simulation pkg is fine now.

File: src/tb3_simulation/urdf/tb3_waffle.urdf (robot description, URDF)
Before this commit: robot turtlebot3_waffle, 13 links, 12 joints
Links:
- link base_link: geometry collision box size=0.266 0.266 0.094; visual mesh filename=/Users/jiteshbhati/Projects/DRL-Turtlebot3/src/tb3_simulati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 scale=0.001 0.001 0.001
- link camera_link: geometry collision box size=0.012 0.132 0.020; visual mesh filename=/Users/jiteshbhati/Projects/DRL-Turtlebot3/src/tb3_simulati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 scale=0.001 0.001 0.001
- link scan_link: geometry collision cylinder length=0.0315 radius=0.055; visual mesh filename=/Users/jiteshbhati/Projects/DRL-Turtlebot3/src/tb3_simulati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 scale=0.001 0.001 0.001
- link wheel_left_link: geometry collision cylinder length=0.018 radius=0.033; visual mesh filename=/Users/jiteshbhati/Projects/DRL-Turtlebot3/src/tb3_simulati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 scale=0.001 0.001 0.001
- link wheel_right_link: geometry collision cylinder length=0.018 radius=0.033; visual mesh filename=/Users/jiteshbhati/Projects/DRL-Turtlebot3/src/tb3_simulati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 scale=0.001 0.001 0.001
